File: projet electronique PCBot/usb.kicad_sch (KiCad schematic)
At the start: 0 parts

Commit message: Ajour USB
Parts:
- added J5: USB_C_Receptacle_USB2.0_16P, Connector_USB:USB_C_Receptacle_GCT_USB4105-xx-A_16P_TopMnt_Horizontal, symbol Connector:USB_C_Receptacle_USB2.0_16P
- added R1, R2: 5k1, Resistor_SMD:R_0402_1005Metric, symbol Device:R_Small
Connections:
- new net: J5.A5 (CC1), R2.1
- new net: J5.B5 (CC2), R1.1
- new net GND: J5.A1 (GND), J5.A12 (GND), J5.B1 (GND), J5.B12 (GND), J5.S1 (SHIELD), R1.2, R2.2
- new net VBUS: J5.A4 (VBUS), J5.A9 (VBUS), J5.B4 (VBUS), J5.B9 (VBUS)
- no-connect marks 0 -> 6
