File: projet electronique PCBot/stm32.kicad_sch (KiCad schematic)
At the start: 8 parts, among them J1 Conn_ST_STDC14, U1 STM32G431KBT6

Commit message: re modification de gestion energie
Parts:
- removed R1, R2: 3.3, symbol Device:R_Small
Connections:
- no-connect marks 2 -> 0

Commit message: stm32
Parts:
- added R1, R2: 3.3, symbol Device:R_Small
Connections:
- net I2C_SCL: now also R1.1
- net I2C_SDA: now also R2.1
- new net: R1.2, R2.2
