File: projet electronique PCBot/stm32.kicad_sch (KiCad schematic)
At the start: 6 parts, among them J1 Conn_ST_STDC14, U1 STM32G431KBT6

Commit message: grosse modif pcb du prof
Parts:
- added C21: 100n, Capacitor_SMD:C_0402_1005Metric, symbol Device:C_Small
- C1, C3, C4: footprint (none) -> Capacitor_SMD:C_0402_1005Metric
- C2: value 200n -> 100n; footprint (none) -> Capacitor_SMD:C_0402_1005Metric
Connections:
- net PG10 is gone; now on net NRST: U1.4 (PG10)
- net +3.3V: now also C21.1
- net GND: now also C21.2
- net USART2_RX: now also J1.13 (VCP_RX); no longer J1.14 (VCP_TX)
- net USART2_TX: now also J1.14 (VCP_TX); no longer J1.13 (VCP_RX), J1.8 (JTDO/SWO)
- no-connect marks 2 -> 3
Other:
- moved on the sheet: C1, C2

Commit message: modif après revu prof
Connections:
- net PA0 renamed TOF3_XSHUT
- net PA1 renamed TOF2_XSHUT
- net PA10 renamed CE
- net PA2 renamed TOF1_XSHUT
- net PA5 renamed SCK
- net PA6 renamed MOSI
- net PA7 renamed MISO
- net PB0 renamed INT
- net PB4 renamed CSN
- net PB5 renamed ~{CE}
- net PB6 renamed IRQ
Other:
- note added: "PF0 PF1 a vérifier"
Changed lines of the file:
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@@
 	(generator_version "9.0")
 	(paper "A4")
+	(text "PF0 PF1 a vérifier\n"
+		(exclude_from_sim no)
+		(at 118.11 88.138 0)
+		(effects
+			(font
+				(size 1.27 1.27)
+			)
+		)
+	)
 	(text "NRST????\n"
 		(exclude_from_sim no)
@@
 		)
 	)
-	(hierarchical_label "PB4"
+	(hierarchical_label "CSN"
 		(shape input)
 		(at 132.08 104.14 180)
@@
 		)
 	)
-	(hierarchical_label "PA0"
+	(hierarchical_label "TOF3_XSHUT"
 		(shape input)
 		(at 157.48 86.36 0)
@@
 		)
 	)
-	(hierarchical_label "PA1"
+	(hierarchical_label "TOF2_XSHUT"
 		(shape input)
 		(at 157.48 88.9 0)
@@
 		)
 	)
-	(hierarchical_label "PB6"
+	(hierarchical_label "IRQ"
 		(shape input)
 		(at 132.08 109.22 180)
@@
 		)
 	)
-	(hierarchical_label "PA6"
+	(hierarchical_label "MOSI"
 		(shape input)
 		(at 157.48 101.6 0)
@@
 		)
 	)
-	(hierarchical_label "PB5"
+	(hierarchical_label "~{CE}"
 		(shape input)
 		(at 132.08 106.68 180)
@@
 		)
 	)
-	(hierarchical_label "PB0"
+	(hierarchical_label "INT"
 		(shape input)
 		(at 132.08 99.06 180)
@@
 		)
 	)
-	(hierarchical_label "PA10"
+	(hierarchical_label "CE"
 		(shape input)
 		(at 157.48 111.76 0)
@@
 		)
 	)
-	(hierarchical_label "PA2"
+	(hierarchical_label "TOF1_XSHUT"
 		(shape input)
 		(at 157.48 91.44 0)
@@
 		)
 	)
-	(hierarchical_label "PA5"
+	(hierarchical_label "SCK"
 		(shape input)
 		(at 157.48 99.06 0)
@@
 		)
 	)
-	(hierarchical_label "PA7"
+	(hierarchical_label "MISO"
 		(shape input)
 		(at 157.48 104.14 0)

Commit message: début routage
Other:
- note added: "PF0 PF1 à vérifier"
- note removed: "NRST????"
- note removed: "PF0 PF1 a vérifier"
Changed lines of the file:
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@@
 	(generator_version "9.0")
 	(paper "A4")
-	(text "PF0 PF1 a vérifier\n"
+	(text "PF0 PF1 à vérifier\n"
 		(exclude_from_sim no)
-		(at 118.11 88.138 0)
-		(effects
-			(font
-				(size 1.27 1.27)
-			)
-		)
-	)
-	(text "NRST????\n"
-		(exclude_from_sim no)
-		(at 81.28 122.682 0)
+		(at 116.84 92.71 0)
 		(effects
 			(font
@@
 		(on_board yes)
 		(dnp no)
-		(fields_autoplaced yes)
 		(property "Reference" "#PWR08"
 			(at 144.78 142.24 0)
@@
 		)
 		(property "Value" "GND"
-			(at 144.78 140.97 0)
-			(effects
-				(font
+			(at 144.78 140.208 0)
+			(effects
+				(font

Commit message: placement sur kicad debut
Connections:
- net PF0: no longer names the net of U1.2 (PF0)
- net PF1: no longer names the net of U1.3 (PF1)
- no-connect marks 3 -> 5
Other:
- note removed: "PF0 PF1 à vérifier"
Changed lines of the file:
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@@
 	(generator_version "9.0")
 	(paper "A4")
-	(text "PF0 PF1 à vérifier\n"
-		(exclude_from_sim no)
-		(at 116.84 92.71 0)
-		(effects
-			(font
-				(size 1.27 1.27)
-			)
-		)
-	)
 	(junction
 		(at 143.51 66.04)
@@
 	)
 	(no_connect
+		(at 132.08 93.98)
+	)
+	(no_connect
 		(at 80.01 107.95)
+	)
+	(no_connect
+		(at 132.08 91.44)
 	)
 	(wire
@@
 		)
 	)
-	(hierarchical_label "PF1"
-		(shape input)
-		(at 132.08 93.98 180)
+	(hierarchical_label "I2C_SDA"
+		(shape input)
+		(at 132.08 111.76 180)
 		(effects
 			(font
@@
 		)
 	)
-	(hierarchical_label "I2C_SDA"
-		(shape input)
-		(at 132.08 111.76 180)
-		(effects
-			(font
-				(size 1.27 1.27)
-			)
-			(justify right)
-		)
-	)
 	(hierarchical_label "TIM1_CH2"
 		(shape input)
@@
 		(effects
 			(font
-				(size 1.27 1.27)
-			)
-			(justify right)
-		)
-	)
-	(hierarchical_label "PF0"
-		(shape input)
-		(at 132.08 91.44 180)
-		(effects
-			(font
