File: projet electronique PCBot/connecteurs.kicad_sch (KiCad schematic)
At the start: 0 parts

Commit message: modif
Parts:
- added Batterie, Moteur, nrf24: Conn_01x02, symbol Connector_Generic:Conn_01x02
Connections:
- new net GND: Batterie.2 (Pin_2), Moteur.2 (Pin_2), nrf24.2 (Pin_2)
- new net Vcc_batt: Batterie.1 (Pin_1)
- new net Vcc_mot: Moteur.1 (Pin_1)
- new net Vcc_nrf: nrf24.1 (Pin_1)

Commit message: connec
Parts:
- added Driver, driver_inertielle, tof: Conn_01x02, symbol Connector_Generic:Conn_01x02
Connections:
- net GND: now also Driver.2 (Pin_2), driver_inertielle.2 (Pin_2), tof.2 (Pin_2)
- new net Vcc_driver: Driver.1 (Pin_1)
- new net Vcc_inert: driver_inertielle.1 (Pin_1)
- new net Vcc_tof: tof.1 (Pin_1)
Other:
- note added: "BMS et Batterie"
- note added: "JST SH"
- note added: "JST VH"
- note added: "driver inertielle et stm32"
- note added: "nrf24 et stm32"
- note added: "sortie régulateur vers driver"
- note added: "sortie régulateur vers moteur"
- note added: "tof et stm32"
- moved on the sheet: Moteur
