File: projet electronique PCBot/capteur.kicad_sch (KiCad schematic)
At the start: 7 parts, among them J1 TOF, J2 TOF, J2 nRF24, J3 TOF, U5 LSM6DSOX

Commit message: modifs
Parts:
- renumbered J1 to J3, J3 to J4, J2 to J6
Connections:
- net VCC is gone; now on net +3.3V: J3.1 (3.3V), J4.1 (3.3V), J6.1 (3.3V)
- net TOF1_GPIO1: no longer names the net of J3.5 (GPIO1)
- net TOF2_GPIO1: no longer names the net of J6.5 (GPIO1)
- net TOF3_GPIO1: no longer names the net of J4.5 (GPIO1)
- no-connect marks 6 -> 9
Other:
- note added: "A vérifier si c'est bien +3.3V pour les TOF (à la place de VCC)"
