File: projet electronique PCBot/capteur.kicad_sch (KiCad schematic)
At the start: 7 parts, among them J2 nRF24, J3 TOF, J4 TOF, J6 TOF, U5 LSM6DSOX

Commit message: grosse modif pcb du prof
Parts:
- added C7: 10u, Capacitor_SMD:C_0603_1608Metric, symbol Device:C_Small
- added C8: 100n, Capacitor_SMD:C_0402_1005Metric, symbol Device:C_Small
- C5, C6: footprint (none) -> Capacitor_SMD:C_0402_1005Metric
- J2: footprint (none) -> Connector_PinSocket_2.54mm:PinSocket_2x04_P2.54mm_Vertical
- J3, J4, J6: footprint (none) -> Connector_PinSocket_2.54mm:PinSocket_1x06_P2.54mm_Vertical
Connections:
- net +3.3V: now also C7.1, C8.1
- net GND: now also C7.2, C8.2
