File: projet electronique PCBot/projet electronique PCBot.kicad_pcb (KiCad board)
At the start: 4 copper layers, 60 x 70 mm, 54 parts, among them J1 Conn_ST_STDC14, J10 Conn_01x02_Pin, J2 nRF24, J3 TOF, J4 TOF, J5 USB_C_Receptacle_USB2.0_16P, J6 TOF, J7 ON SWITCH, J8 Conn_01x02_Pin, J9 Conn_01x02_Pin, U1 STM32G431KBT6, U2 BQ25896RTWR, U3 BU33SD5WG-TR, U4 DRV8411APWPR, U5 LSM6DSOX

Commit message: début routage
Parts:
- added H1: MountingHole_Pad, MountingHole:MountingHole_3.2mm_M3_DIN965_Pad, F.Cu at (115.0, 35.0)
- added H2: MountingHole_Pad, MountingHole:MountingHole_3.2mm_M3_DIN965_Pad, F.Cu at (165.0, 35.0)
- added H3: MountingHole_Pad, MountingHole:MountingHole_3.2mm_M3_DIN965_Pad, F.Cu at (115.0, 95.0)
- added H4: MountingHole_Pad, MountingHole:MountingHole_3.2mm_M3_DIN965_Pad, F.Cu at (165.0, 95.0)
- moved C1 9.05 mm to (159.6, 53.0)
- moved C2 9.05 mm to (159.6, 54.9)
- moved C21 9.05 mm to (159.6, 60.8)
- moved C3 9.05 mm to (159.6, 56.9)
- moved C4 9.05 mm to (159.6, 58.9)
- moved J1 9.05 mm to (163.0, 46.5)
Connections:
- net /Driver/PA4 renamed /Driver/nFAULT
- net /PA4 renamed /STM32/PA4
- net /STM32/PA1 renamed /TOF1_XSHUT
- net /STM32/PA2 renamed /STM32/TOF1_XSHUT
- net /STM32/TIM1_CH1 renamed /TIM1_CH1
- net /STM32/TIM1_CH1N renamed /TIM1_CH1N
- net /STM32/TIM1_CH2 renamed /TIM1_CH2
- net /STM32/TIM1_CH2N renamed /TIM1_CH2N
- net /TOF2_XSHUT renamed /STM32/PF0
- U1 pad 3: /TOF3_XSHUT -> /STM32/PF1
- U1 pad 5: /STM32/PA0 -> /TOF3_XSHUT
- U4 pad 10: unconnected-(U4-BIN2-Pad10) -> /Driver/TIM1_CH2N
- U4 pad 15: unconnected-(U4-AIN2-Pad15) -> /Driver/TIM1_CH1N
- U4 pad 16: unconnected-(U4-AIN1-Pad16) -> /Driver/TIM1_CH1
- U4 pad 9: unconnected-(U4-BIN1-Pad9) -> /Driver/TIM1_CH2
Routing:
- added copper zone on B.Cu, net GND
- added copper zone on F.Cu, net GND
Other:
- outline, holes or cut-outs redrawn

Commit message: placement sur kicad debut
Parts:
- moved U1 18.2 mm to (140.1, 63.8)
- moved R2 9.63 mm to (129.9, 97.8)
- moved R1 9.63 mm to (129.9, 95.8)
- moved C18 7.90 mm to (150.7, 82.0)
- moved R11 7.90 mm to (147.8, 79.0)
- moved R12 7.90 mm to (147.8, 81.0)
- moved U4 7.90 mm to (151.2, 74.7)
- moved C20 7.90 mm to (151.5, 79.5)
- moved J10 7.90 mm to (140.4, 82.6)
- moved J9 7.90 mm to (140.4, 74.8)
- moved J5 7.64 mm to (137.9, 91.9)
- moved R13 6.81 mm to (148.5, 81.9)
- moved U3 6.81 mm to (156.3, 85.7)
- moved D2 4.35 mm to (135.9, 78.7)
- moved D1 4.35 mm to (135.9, 76.2)
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Routing:
- net +3.3V: track 0.00 -> 2.68 mm, vias 2 -> 18
- net GND: track 0.00 -> 0.52 mm, vias 1 -> 46

Commit message: suite placement composants
Parts:
- JP1, JP2: moved to B.Cu
- moved J6 42.5 mm to (166.0, 57.7)
- moved C17 36.2 mm to (154.0, 70.5)
- moved C16 34.4 mm to (153.5, 75.8)
- moved R3 26.5 mm to (137.9, 79.9)
- moved U5 25.8 mm to (140.0, 46.9)
- moved R5 24.7 mm to (140.8, 71.4)
- moved C1 24.7 mm to (135.0, 54.5)
- moved R6 24.6 mm to (140.8, 72.9)
- moved C2 24.6 mm to (135.0, 55.5)
- moved J10 24.2 mm to (164.0, 88.2), turned to 90 degrees
- moved J9 23.9 mm to (164.0, 78.8), turned to 90 degrees
- moved R4 22.7 mm to (137.4, 74.9)
- moved J2 21.5 mm to (112.9, 48.7), turned to 180 degrees
- moved C3 20.3 mm to (141.5, 66.0), turned to 180 degrees
- moved C4 19.9 mm to (141.5, 67.0), turned to 180 degrees
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Connections:
- net Net-(C10-Pad1) renamed /Gestion d'energie/SW
- R5 pad 1: Net-(R5-Pad1) -> +3.3V
- R6 pad 1: Net-(R5-Pad1) -> +3.3V
- R8 pad 1: Net-(R5-Pad1) -> +3.3V
- U1 pad 2: /STM32/PF0 -> unconnected-(U1-PF0-Pad2)
- U1 pad 3: /STM32/PF1 -> unconnected-(U1-PF1-Pad3)
- U4 pad 5: Net-(J9-Pin_2) -> Net-(J9-Pin_1)
- U4 pad 7: Net-(J9-Pin_1) -> Net-(J9-Pin_2)
Routing:
- net GND: track 0.52 -> 4.75 mm, vias 46 -> 3
- net +3.3V: track 2.68 -> 0.00 mm, vias 18 -> 1
- net /Gestion d'energie/SYS: vias 2 -> 0
- added copper zone on F.Cu, net /Gestion d'energie/SW
- added copper zone on F.Cu, net Net-(JP2-A)

Commit message: routage avec bcp d'erreurs
Parts:
- moved J4 16.0 mm to (146.7, 33.4), turned to -90 degrees
- moved J3 11.1 mm to (113.0, 69.1), turned to 180 degrees
- moved D2 10.2 mm to (145.8, 75.4)
- moved D1 8.65 mm to (145.8, 78.8)
- moved R2 3.51 mm to (130.5, 89.3), turned to 90 degrees
- moved C19 2.89 mm to (150.2, 84.2), turned to -90 degrees
- moved R12 2.76 mm to (147.8, 86.7), turned to 0 degrees
- moved R1 2.53 mm to (133.5, 89.3)
- moved R11 2.41 mm to (147.7, 81.9)
- moved J1 1.88 mm to (164.2, 45.0), turned to 180 degrees
- moved JP1 1.63 mm to (138.8, 76.9)
- moved C5 0.31 mm to (138.8, 48.9)
- moved C20 0.28 mm to (147.7, 84.3), turned to -90 degrees
- turned R3 to 180 degrees
- turned R5 to 180 degrees
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Connections:
- C19 pad 1: /Driver/SYS -> /Gestion d'energie/SYS
- C20 pad 1: /Driver/SYS -> /Gestion d'energie/SYS
- J5 pad A4: VBUS -> /Gestion d'energie/VBUS
- J5 pad A9: VBUS -> /Gestion d'energie/VBUS
- J5 pad B4: VBUS -> /Gestion d'energie/VBUS
- J5 pad B9: VBUS -> /Gestion d'energie/VBUS
- R5 pad 2: /Gestion d'energie/SDA -> /Capteur/SDA
- R6 pad 2: /Gestion d'energie/SCL -> /Capteur/SCL
- U1 pad 10: /SCK -> /Capteur/SCK
- U1 pad 11: /MOSI -> /Capteur/MOSI
- U1 pad 12: /MISO -> /Capteur/MISO
- U1 pad 13: /INT -> /Gestion d'energie/INT
- U1 pad 18: /TIM1_CH1 -> /Driver/TIM1_CH1
- U1 pad 19: /TIM1_CH2 -> /Driver/TIM1_CH2
- U1 pad 20: /CE -> /Capteur/CE
- U1 pad 21: /TIM1_CH1N -> /Driver/TIM1_CH1N
- U1 pad 22: /TIM1_CH2N -> /Driver/TIM1_CH2N
- U1 pad 27: /CSN -> /Capteur/CSN
- U1 pad 28: /~{CE} -> /Gestion d'energie/~{CE}
- U1 pad 29: /IRQ -> /Capteur/IRQ
- U1 pad 30: /SDA -> /Capteur/SDA
- U1 pad 31: /SCL -> /Capteur/SCL
- U1 pad 5: /TOF3_XSHUT -> /Capteur/TOF3_XSHUT
- U1 pad 6: /TOF1_XSHUT -> /Capteur/TOF2_XSHUT
- U1 pad 7: /STM32/TOF1_XSHUT -> /Capteur/TOF1_XSHUT
- U2 pad 5: /Gestion d'energie/SCL -> /Capteur/SCL
- U2 pad 6: /Gestion d'energie/SDA -> /Capteur/SDA
- U4 pad 12: /Driver/SYS -> /Gestion d'energie/SYS
Routing:
- net /Capteur/SDA: track 0.00 -> 180.7 mm, vias 0 -> 3
- net /Capteur/SCL: track 0.00 -> 131.4 mm, vias 0 -> 2
- net /STM32/NRST: track 0.00 -> 74.9 mm, vias 0 -> 3
- net /Capteur/CE: track 0.00 -> 46.1 mm, vias 0 -> 5
- net /Capteur/TOF2_XSHUT: track 0.00 -> 41.8 mm, vias 0 -> 2
- net /Capteur/MISO: track 0.00 -> 40.3 mm, vias 0 -> 2
- net /Capteur/CSN: track 0.00 -> 40.2 mm, vias 0 -> 1
- net /Gestion d'energie/~{CE}: track 0.00 -> 40.1 mm, vias 0 -> 7
- net /Capteur/TOF3_XSHUT: track 0.00 -> 38.8 mm, vias 0 -> 2
- net /Capteur/SCK: track 0.00 -> 36.2 mm, vias 0 -> 2
- net /Gestion d'energie/SYS: track 0.00 -> 36.1 mm, vias 0 -> 8
- net /Capteur/MOSI: track 0.00 -> 36.1 mm, vias 0 -> 2
- net /Capteur/IRQ: track 0.00 -> 30.6 mm, vias 0 -> 1
- net /STM32/USART2_RX: track 0.00 -> 30.0 mm
- net /Driver/TIM1_CH1N: track 0.00 -> 29.6 mm, vias 0 -> 1
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