File: projet electronique PCBot/projet electronique PCBot.kicad_pcb (KiCad board)
At the start: 4 copper layers, 60 x 70 mm, 58 parts, among them J1 Conn_ST_STDC14, J10 Conn_01x02_Pin, J2 nRF24, J3 TOF, J4 TOF, J5 USB_C_Receptacle_USB2.0_16P, J6 TOF, J7 ON SWITCH, J8 Conn_01x02_Pin, J9 Conn_01x02_Pin, U1 STM32G431KBT6, U2 BQ25896RTWR, U3 BU33SD5WG-TR, U4 DRV8411APWPR, U5 LSM6DSOX

Commit message: routage avec 30 erreurs
Parts:
- moved R12 1.10 mm to (147.7, 87.8)
- moved C20 0.65 mm to (147.1, 84.5)
- moved C16 0.44 mm to (153.5, 76.2)
- moved U3 0.40 mm to (154.1, 73.5)
Routing:
- net /Gestion d'energie/SW: track 0.00 -> 10.3 mm
- net Net-(JP2-A): track 4.82 -> 13.7 mm
- net /Driver/TIM1_CH1N: track 29.6 -> 34.6 mm, vias 1 -> 2
- net /Capteur/SDA: track 180.7 -> 183.5 mm, vias 3 -> 4
- net /Driver/TIM1_CH1: track 28.0 -> 30.6 mm, vias 1 -> 2
- net /Capteur/SCL: track 131.4 -> 133.7 mm, vias 2 -> 3
- net /Driver/TIM1_CH2N: track 27.9 -> 30.1 mm
- net /Gestion d'energie/VBUS: track 27.6 -> 26.4 mm, vias 0 -> 1
- net /Capteur/IRQ: track 30.6 -> 31.5 mm, vias 1 -> 2
- net Net-(U4-AIPROPI): track 4.50 -> 5.21 mm
- net /Gestion d'energie/SYS: track 36.1 -> 36.6 mm, vias 8 -> 7
- net GND: track 2.83 -> 3.21 mm, vias 45 -> 57
- net /Capteur/CE: track 46.1 -> 46.4 mm, vias 5 -> 6
- net /Capteur/CSN: track 40.2 -> 40.1 mm, vias 1 -> 2
- net Net-(J9-Pin_2): track 10.7 -> 10.6 mm, vias 1 -> 2
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
Commit message: modif routage fin
Parts:
- moved JP1 10.1 mm to (136.3, 86.7), turned to 90 degrees
- moved R13 3.68 mm to (157.8, 79.8), turned to -90 degrees
- moved JP2 2.90 mm to (122.0, 76.8), turned to -90 degrees
Connections:
- net Net-(J10-Pin_1) renamed /Driver/AOUT1
- net Net-(J10-Pin_2) renamed /Driver/AOUT2
- net Net-(J9-Pin_1) renamed /Driver/BOUT2
- net Net-(J9-Pin_2) renamed /Driver/BOUT1
- net Net-(JP1-B) renamed /Gestion d'energie/VBUS_TO_BQ
Routing:
- net /Gestion d'energie/SYS: track 36.6 -> 5.11 mm, vias 7 -> 9
- net /Gestion d'energie/VBUS: track 26.4 -> 0.00 mm, vias 1 -> 4
- net Net-(JP2-A): track 13.7 -> 0.00 mm, vias 0 -> 2
- net /Driver/BOUT1: track 10.6 -> 0.00 mm, vias 2 -> 0
- net /Gestion d'energie/SW: track 10.3 -> 0.00 mm
- net Net-(U2-REGN): track 1.87 -> 11.7 mm, vias 0 -> 2
- net /Driver/BOUT2: track 9.76 -> 0.00 mm
- net /Driver/AOUT1: track 7.16 -> 0.00 mm
- net /Driver/AOUT2: track 6.66 -> 0.00 mm
- net GND: track 3.21 -> 7.41 mm, vias 57 -> 53
- net +3.3V: track 2.29 -> 6.06 mm, vias 21 -> 22
- net /Gestion d'energie/INT: track 11.6 -> 13.4 mm
- net Net-(U2-ILIM): track 0.00 -> 1.76 mm
- net /Capteur/SDA: track 183.5 -> 182.6 mm
- net /Driver/nFAULT: track 2.47 -> 1.55 mm
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- added copper zone on F.Cu, net /Driver/BOUT1
- added copper zone on In2.Cu, net /Gestion d'energie/VBUS
- added copper zone on F.Cu, net /Gestion d'energie/VBUS_TO_BQ

Commit message: routageee
Routing:
- added copper zone on F.Cu, net /Driver/AOUT1
- added copper zone on F.Cu, net /Driver/AOUT2
- added copper zone on F.Cu, net /Driver/BOUT2
Changed lines of the file:
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@@
 		)
 		(fp_text user "${REFERENCE}"
-			(at 0 0 0)
+			(at 0.1375 0 0)
 			(layer "F.Fab")
 			(effects
@@
 		(tags "resistor")
 		(property "Reference" "R13"
-			(at 1.65 -0.68 0)
+			(at 0.6 3.6 0)
 			(layer "F.SilkS")
 			(effects
@@
 		)
 		(property "Value" "10u"
-			(at 0 1.43 90)
+			(at 1.3 1.6 90)
 			(layer "F.Fab")
 			(effects
@@
 		)
 		(property "Value" "DRV8411APWPR"
-			(at 0 3.45 0)
+			(at 0.2 -7.5 0)
 			(layer "F.Fab")
 			(effects
@@
 		(tags "USB C Type-C Receptacle SMD USB 2.0 16P 16C USB4105-15-A USB4105-15-A-060 USB4105-15-A-120 USB4105-GF-A USB4105-GF-A-060 USB4105-GF-A-120")
 		(property "Reference" "J5"
-			(at -2.26 -2.22 0)
+			(at -2.95 -0.78 0)
 			(unlocked yes)
 			(layer "F.SilkS")
@@
 		)
 		(property "Value" "100n"
-			(at 2.98 -0.5 90)
+			(at 3 0 90)
 			(layer "F.Fab")
 			(effects
@@
 		(tags "capacitor")
 		(property "Reference" "C1"
-			(at 0 -1.16 0)
+			(at -2.2 -0.3 0)
 			(layer "F.SilkS")
 			(effects
@@
 		)
 		(property "Value" "4.7u"
-			(at 0 1.16 0)
+			(at 0 -1.1 0)
 			(layer "F.Fab")
 			(effects
@@
 		(tags "capacitor")
 		(property "Reference" "C2"
-			(at 0 -1.16 0)
+			(at -2.22 -0.1 0)
 			(layer "F.SilkS")
 			(effects
@@
 		)
 		(property "Value" "100n"
-			(at 0 1.16 0)
+			(at -2.22 1.5 0)
 			(layer "F.Fab")
 			(effects
@@
 		(tags "Texas WQFN NoLead")
 		(property "Reference" "U2"
-			(at 3.975 -5.375 0)
+			(at 3.375 -5.775 0)
 			(layer "F.SilkS")
 			(effects
@@
 		(tags "inductor")
 		(property "Reference" "L1"
-			(at 0 -2.05 90)
+			(at -2.8 -0.2 90)
 			(layer "F.SilkS")
 			(effects
@@
 		)
 		(property "Value" "1u"
-			(at 0 1.16 0)
+			(at 0 -2.5 0)
 			(layer "F.Fab")
 			(effects
@@
 		)
 		(property "Value" "SolderJumper_2_Open"
-			(at 0 -1.9 90)
+			(at 9.2 -2.4 90)
 			(layer "B.Fab")
 			(effects
@@
 	)
 	(zone
+		(net 43)
+		(net_name "/Driver/BOUT2")
+		(layer "F.Cu")
+		(hatch edge 0.5)
+		(priority 9)
+		(connect_pads yes
+			(clearance 0.2)
+		)
+		(min_thickness 0.25)
+		(filled_areas_thickness no)
+		(fill yes
+			(thermal_gap 0.3)
+			(thermal_bridge_width 0.3)
+		)
+		(polygon
+			(pts
+				(xy 157 84) (xy 161 84) (xy 164.4 83.4) (xy 165 81.8) (xy 165 80.6) (xy 165 79.6) (xy 165 78) (xy 163 78)
+				(xy 163 79.6) (xy 162.4 82.8) (xy 160 83.6) (xy 157 83.6)
+			)
+		)
+	)
+	(zone
+		(net 46)
+		(net_name "/Driver/AOUT2")
+		(layer "F.Cu")
+		(hatch edge 0.5)
+		(priority 9)
+		(connect_pads yes
+			(clearance 0.2)
+		)
+		(min_thickness 0.25)
+		(filled_areas_thickness no)
+		(fill yes
+			(thermal_gap 0.3)
+			(thermal_bridge_width 0.3)
+		)
+		(polygon
+			(pts
+				(xy 156.945205 84.679452) (xy 160.8 84.8) (xy 163.6 86.8) (xy 165 86.8) (xy 165.2 84.8) (xy 163 84.6)
+				(xy 159.945205 84.279452) (xy 156.945205 84.279452)
+			)
+		)
+	)
+	(zone
 		(net 2)
 		(net_name "GND")
@@
 			)
 		)
+	)
+	(zone
+		(net 45)
+		(net_name "/Driver/AOUT1")
+		(layer "F.Cu")
+		(hatch edge 0.5)
+		(priority 9)
+		(connect_pads yes
+			(clearance 0.2)
+		)
+		(min_thickness 0.25)
+		(filled_areas_thickness no)
+		(fill yes
+			(thermal_gap 0.3)
+			(thermal_bridge_width 0.3)
+		)
+		(polygon
+			(pts
+				(xy 157.2 86) (xy 159.6 86) (xy 162.8 89.2) (xy 165.2 89.2) (xy 165.2 87.2) (xy 163 87.2) (xy 160 85.6)
+				(xy 157.2 85.6)
+			)
+		)

Commit message: Dernières corrections LFiack
Parts:
- moved C15 0.28 mm to (114.0, 77.5), turned to 180 degrees
Routing:
- net Net-(J8-Pin_1): track 25.6 -> 0.00 mm
- net /Capteur/SCL: track 133.7 -> 132.2 mm
- added copper zone on F.Cu, net Net-(J8-Pin_1)
