File: projet electronique PCBot/projet electronique PCBot.kicad_sch (KiCad schematic)
At the start: 0 parts

Commit message: modif un lundi lambda
Changed lines of the file:
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@@
+	(wire
+		(pts
+			(xy 204.47 109.22) (xy 222.25 109.22)
+		)
+		(stroke
+			(width 0)
+			(type default)
+		)
+	)
+	(wire
+		(pts
+			(xy 207.01 60.96) (xy 222.25 60.96)
+		)
+		(stroke
+			(width 0)
+			(type default)
+		)
+	)
 	(wire
 		(pts
@@
 	(wire
 		(pts
+			(xy 148.59 97.79) (xy 128.27 97.79)
+		)
+		(stroke
+			(width 0)
+			(type default)
+		)
+	)
+	(wire
+		(pts
 			(xy 85.09 123.19) (xy 85.09 147.32)
 		)
@@
 	(wire
 		(pts
-			(xy 207.01 53.34) (xy 228.6 53.34)
-		)
-		(stroke
-			(width 0)
-			(type default)
-		)
-	)
-	(wire
-		(pts
 			(xy 204.47 104.14) (xy 213.36 104.14)
 		)
@@
 	(wire
 		(pts
+			(xy 207.01 53.34) (xy 227.33 53.34)
+		)
+		(stroke
+			(width 0)
+			(type default)
+		)
+	)
+	(wire
+		(pts
 			(xy 134.62 128.27) (xy 143.51 128.27)
 		)
@@
 	(wire
 		(pts
-			(xy 231.14 111.76) (xy 204.47 111.76)
+			(xy 207.01 63.5) (xy 224.79 63.5)
 		)
 		(stroke
@@
 	(wire
 		(pts
+			(xy 231.14 50.8) (xy 207.01 50.8)
+		)
+		(stroke
+			(width 0)
+			(type default)
+		)
+	)
+	(wire
+		(pts
+			(xy 231.14 29.21) (xy 231.14 50.8)
+		)
+		(stroke
+			(width 0)
+			(type default)
+		)
+	)
+	(wire
+		(pts
+			(xy 148.59 102.87) (xy 124.46 102.87)
+		)
+		(stroke
+			(width 0)
+			(type default)
+		)
+	)
+	(wire
+		(pts
 			(xy 162.56 48.26) (xy 140.97 48.26)
 		)
@@
 	(wire
 		(pts
-			(xy 231.14 50.8) (xy 231.14 111.76)
-		)
-		(stroke
-			(width 0)
-			(type default)
-		)
-	)
-	(wire
-		(pts
-			(xy 207.01 50.8) (xy 231.14 50.8)
+			(xy 227.33 31.75) (xy 227.33 53.34)
 		)
 		(stroke
@@
 	(wire
 		(pts
+			(xy 129.54 31.75) (xy 227.33 31.75)
+		)
+		(stroke
+			(width 0)
+			(type default)
+		)
+	)
+	(wire
+		(pts
+			(xy 124.46 29.21) (xy 231.14 29.21)
+		)
+		(stroke
+			(width 0)
+			(type default)
+		)
+	)
+	(wire
+		(pts
 			(xy 213.36 74.93) (xy 38.1 74.93)
 		)
@@
 	(wire
 		(pts
-			(xy 228.6 53.34) (xy 228.6 109.22)
-		)
-		(stroke
-			(width 0)
-			(type default)
-		)
-	)
-	(wire
-		(pts
 			(xy 140.97 48.26) (xy 140.97 125.73)
 		)
@@
 	(wire
 		(pts
+			(xy 222.25 35.56) (xy 222.25 48.26)
+		)
+		(stroke
+			(width 0)
+			(type default)
+		)
+	)
+	(wire
+		(pts
 			(xy 215.9 38.1) (xy 215.9 106.68)
 		)
@@
 	(wire
 		(pts
-			(xy 220.98 64.77) (xy 220.98 116.84)
+			(xy 220.98 66.04) (xy 220.98 116.84)
+		)
+		(stroke
+			(width 0)
+			(type default)
+		)
+	)
+	(wire
+		(pts
+			(xy 224.79 63.5) (xy 224.79 111.76)
 		)
 		(stroke
@@
 	(wire
 		(pts
-			(xy 233.68 48.26) (xy 233.68 114.3)
+			(xy 124.46 102.87) (xy 124.46 29.21)
+		)
+		(stroke
+			(width 0)
+			(type default)
+		)
+	)
+	(wire
+		(pts
+			(xy 207.01 58.42) (xy 226.06 58.42)
 		)
 		(stroke
@@
 	(wire
 		(pts
-			(xy 207.01 48.26) (xy 233.68 48.26)
+			(xy 148.59 105.41) (xy 129.54 105.41)
 		)
 		(stroke
@@
 	(wire
 		(pts
-			(xy 228.6 109.22) (xy 204.47 109.22)
+			(xy 129.54 105.41) (xy 129.54 31.75)
 		)
 		(stroke
@@
 	(wire
 		(pts
+			(xy 222.25 48.26) (xy 207.01 48.26)
+		)
+		(stroke
+			(width 0)
+			(type default)
+		)
+	)
+	(wire
+		(pts
 			(xy 93.98 130.81) (xy 90.17 130.81)
 		)
@@
 	(wire
 		(pts
-			(xy 207.01 64.77) (xy 220.98 64.77)
+			(xy 224.79 111.76) (xy 204.47 111.76)
+		)
+		(stroke
+			(width 0)
+			(type default)
+		)
+	)
+	(wire
+		(pts
+			(xy 207.01 66.04) (xy 220.98 66.04)
+		)
+		(stroke
+			(width 0)
+			(type default)
+		)
+	)
+	(wire
+		(pts
+			(xy 128.27 35.56) (xy 222.25 35.56)
+		)
+		(stroke
+			(width 0)
+			(type default)
+		)
+	)
+	(wire
+		(pts
+			(xy 226.06 58.42) (xy 226.06 114.3)
 		)
 		(stroke
@@
 	(wire
 		(pts
+			(xy 222.25 60.96) (xy 222.25 109.22)
+		)
+		(stroke
+			(width 0)
+			(type default)
+		)
+	)
+	(wire
+		(pts
 			(xy 88.9 143.51) (xy 129.54 143.51)
 		)
@@
 	(wire
 		(pts
-			(xy 233.68 114.3) (xy 204.47 114.3)
+			(xy 226.06 114.3) (xy 204.47 114.3)
+		)
+		(stroke
+			(width 0)
+			(type default)
+		)
+	)
+	(wire
+		(pts
+			(xy 128.27 97.79) (xy 128.27 35.56)
 		)
 		(stroke
@@
 		)
 	)
-	(hierarchical_label "PA0"
+	(hierarchical_label "PA4"
 		(shape input)
 		(at 91.44 41.91 270)
@@
 		)
 	)
+	(hierarchical_label "MOSI"
+		(shape input)
+		(at 207.01 63.5 180)
+		(effects
+			(font
+				(size 1.27 1.27)
+			)
+			(justify right)
+		)
+	)
 	(hierarchical_label "INT"
 		(shape input)
@@
 	(hierarchical_label "CE"
 		(shape input)
-		(at 207.01 64.77 180)
+		(at 207.01 66.04 180)
 		(effects
 			(font
@@
 		)
 	)
+	(hierarchical_label "SCK"
+		(shape input)
+		(at 207.01 58.42 180)
+		(effects
+			(font
+				(size 1.27 1.27)
+			)
+			(justify right)
+		)
+	)
 	(hierarchical_label "IRQ"
 		(shape input)
@@
 		)
 	)
+	(hierarchical_label "MISO"
+		(shape input)
+		(at 207.01 60.96 180)
+		(effects
+			(font
+				(size 1.27 1.27)
+			)
+			(justify right)
+		)
+	)

Commit message: re modif de lundi
Other:
- sheet STM32 ports: added none; removed SWDIO, SWO, VCC, VCP_RX, VCP_TX, ~{RST}
Changed lines of the file:
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@@
-			)
-		)
-		(pin "SWDIO" input
-			(at 172.72 87.63 90)
-			(effects
-				(font
-					(size 1.27 1.27)
-				)
-				(justify right)
-			)
-		)
-		(pin "SWO" input
-			(at 175.26 87.63 90)
-			(effects
-				(font
-					(size 1.27 1.27)
-				)
-				(justify right)
 			)
 		)
@@
 			)
 		)
-		(pin "VCC" input
-			(at 165.1 87.63 90)
-			(effects
-				(font
-					(size 1.27 1.27)
-				)
-				(justify right)
-			)
-		)
-		(pin "VCP_RX" input
-			(at 179.07 87.63 90)
-			(effects
-				(font
-					(size 1.27 1.27)
-				)
-				(justify right)
-			)
-		)
-		(pin "VCP_TX" input
-			(at 181.61 87.63 90)
-			(effects
-				(font
-					(size 1.27 1.27)
-				)
-				(justify right)
-			)
-		)
-		(pin "~{RST}" input
-			(at 167.64 87.63 90)
-			(effects
-				(font
-					(size 1.27 1.27)
-				)
-				(justify right)
-			)
-		)

Commit message: grosse modif pcb du prof
Other:
- note added: "Vers AINX du driver"

Commit message: modif après revu prof
Other:
- sheet STM32 ports: added CE, CSN, INT, IRQ, MISO, MOSI, SCK, TOF2_XSHUT, TOF3_XSHUT, nFAULT, ~{CE}; removed PA0, PA1, PA10, PA2, PA4, PA5, PA6, PA7, PB0, PB4, PB5, PB6

Commit message: début routage
Parts:
- added H1, H2, H3, H4: MountingHole_Pad, MountingHole:MountingHole_3.2mm_M3_DIN965_Pad, symbol Mechanical:MountingHole_Pad
Connections:
- new net GND: H1.1, H2.1, H3.1, H4.1
Other:
- note removed: "Vers AINX du driver"

Commit message: routage avec bcp d'erreurs
Other:
- sheet Capteur ports: added CE, CSN, IRQ, MISO, MOSI, SCK, SCL, SDA, TOF1_XSHUT, TOF2_XSHUT, TOF3_XSHUT; removed none
- sheet Driver ports: added SYS, TIM1_CH1, TIM1_CH1N, TIM1_CH2, TIM1_CH2N, nFAULT; removed none
- sheet Gestion d'energie ports: added INT, OTG, SCL, SDA, SYS, VBUS, ~{CE}; removed none
- sheet STM32 ports: added PA4, TOF1_XSHUT; removed none
- sheet USB ports: added VBUS; removed none
