File: projet electronique PCBot/driver.kicad_sch (KiCad schematic)
At the start: 9 parts, among them U4 DRV8833PWP

Commit message: modif un lundi lambda
Connections:
- net PA0: no longer R?.1
- new net PA4: R?.1
Changed lines of the file:
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@@
 		)
 	)
-	(hierarchical_label "PA0"
+	(hierarchical_label "PA4"
 		(shape input)
 		(at 154.94 88.9 90)

Commit message: grosse modif pcb du prof
Parts:
- C18: renamed from C?; footprint (none) -> Capacitor_SMD:C_0402_1005Metric
- C19: renamed from C?; value 0u1 -> 100n; footprint (none) -> Capacitor_SMD:C_0402_1005Metric
- C20: renamed from C?; footprint (none) -> Capacitor_SMD:C_0805_2012Metric
- J10, J9: renamed from J?; footprint (none) -> Connector_JST:JST_XH_B2B-XH-A_1x02_P2.50mm_Vertical
- R11, R12, R13: renamed from R?; footprint (none) -> Resistor_SMD:R_0402_1005Metric
- U4: value DRV8833PWP -> DRV8411APWPR
Connections:
- net +3.3V: now also R13.1
- net PA4: now also R13.2, U4.8 (nFAULT); no longer R13.1
- net PA0: no longer names the net of U4.16 (AIN1)
- net PA1: no longer names the net of U4.15 (AIN2)
- net PA2: no longer names the net of U4.9 (BIN1)
- net PA3: no longer names the net of U4.10 (BIN2)
Other:
- note added: "TIMER CHANNEL 1, 1N"
- note added: "TIMER CHANNEL 2, 2N"
Changed lines of the file:
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@@
 	(generator_version "9.0")
 	(paper "A4")
+	(text "TIMER CHANNEL 1, 1N"
+		(exclude_from_sim no)
+		(at 85.09 108.458 0)
+		(effects
+			(font
+				(size 1.27 1.27)
+			)
+		)
+	)
+	(text "TIMER CHANNEL 2, 2N"
+		(exclude_from_sim no)
+		(at 85.09 114.046 0)
+		(effects
+			(font
+				(size 1.27 1.27)
+			)
+		)
+	)
 	(junction
 		(at 107.95 132.08)
@@
 	)
 	(junction
+		(at 154.94 102.87)
+		(diameter 0)
+		(color 0 0 0 0)
+	)
+	(junction
 		(at 118.11 60.96)
 		(diameter 0)
@@
 	(wire
 		(pts
+			(xy 154.94 102.87) (xy 158.75 102.87)
+		)
+		(stroke
+			(width 0)
+			(type default)
+		)
+	)
+	(wire
+		(pts
 			(xy 176.53 90.17) (xy 195.58 90.17)
 		)
@@
 		)
 	)
-	(hierarchical_label "PA1"
+	(hierarchical_label "PA4"
 		(shape input)
-		(at 119.38 110.49 180)
+		(at 158.75 102.87 0)
 		(effects
 			(font
 				(size 1.27 1.27)
 			)
-			(justify right)
-		)
-	)
-	(hierarchical_label "PA4"
+			(justify left)
+		)
+	)
+	(hierarchical_label "TIM1_CH1"
 		(shape input)
-		(at 154.94 88.9 90)
+		(at 102.87 106.68 0)
 		(effects
 			(font
@@
 		)
 	)
-	(hierarchical_label "PA0"
+	(hierarchical_label "TIM1_CH2"
 		(shape input)
-		(at 119.38 107.95 180)
+		(at 102.87 109.22 0)
 		(effects
 			(font
 				(size 1.27 1.27)
 			)
-			(justify right)
-		)
-	)
-	(hierarchical_label "PA3"
-		(shape input)
-		(at 119.38 115.57 180)
-		(effects
-			(font
-				(size 1.27 1.27)
-			)
-			(justify right)
-		)
-	)
-	(hierarchical_label "PA2"
-		(shape input)
-		(at 119.38 113.03 180)
-		(effects
-			(font
-				(size 1.27 1.27)
-			)
-			(justify right)
+			(justify left)
 		)
 	)
@@
 		)
 	)
+	(hierarchical_label "TIM1_CH2N"
+		(shape input)
+		(at 102.87 116.84 0)
+		(effects
+			(font
+				(size 1.27 1.27)
+			)
+			(justify left)
+		)
+	)
+	(hierarchical_label "TIM1_CH1N"
+		(shape input)
+		(at 102.87 114.3 0)
+		(effects
+			(font
+				(size 1.27 1.27)
+			)
+			(justify left)
+		)
+	)
 	(symbol
 		(lib_id "Connector:Conn_01x02_Pin")
@@
 		(dnp no)
 		(fields_autoplaced yes)
-		(property "Reference" "J?"
+		(property "Reference" "J9"
 			(at 188.595 106.68 0)
 			(effects
@@
 			)
 		)
-		(property "Footprint" ""
+		(property "Footprint" "Connector_JST:JST_XH_B2B-XH-A_1x02_P2.50mm_Vertical"
 			(at 187.96 111.76 0)
 			(effects
@@
 			(project "projet electronique PCBot"
 				(path "/210be09d-86cd-4faa-bb91-cc54c5972517/8074907f-d1dc-4b1d-805f-91e9bac82bf7"
-					(reference "J?")
+					(reference "J9")
 					(unit 1)
 				)
@@
 		(dnp no)
 		(fields_autoplaced yes)
-		(property "Reference" "#PWR?"
+		(property "Reference" "#PWR0112"
 			(at 154.94 82.55 0)
 			(effects
@@
 			(project "projet electronique PCBot"
 				(path "/210be09d-86cd-4faa-bb91-cc54c5972517/8074907f-d1dc-4b1d-805f-91e9bac82bf7"
-					(reference "#PWR?")
+					(reference "#PWR0112")
 					(unit 1)
 				)
@@
 		(on_board yes)
 		(dnp no)
-		(property "Reference" "C?"
+		(property "Reference" "C19"
 			(at 157.48 64.7762 0)
 			(effects
@@
 			)
 		)
-		(property "Value" "0u1"
+		(property "Value" "100n"
 			(at 157.48 67.3162 0)
 			(effects
@@
 			)
 		)
-		(property "Footprint" ""
+		(property "Footprint" "Capacitor_SMD:C_0402_1005Metric"
 			(at 154.94 66.04 0)
 			(effects
@@
 			(project "projet electronique PCBot"
 				(path "/210be09d-86cd-4faa-bb91-cc54c5972517/8074907f-d1dc-4b1d-805f-91e9bac82bf7"
-					(reference "C?")
+					(reference "C19")
 					(unit 1)
 				)
@@
 				(path "/7d11412a-f71f-4764-add7-c39197843588"
 					(reference "C1")
+					(unit 1)
+				)
+			)
+		)
+	)
+	(symbol
+		(lib_id "power:+3.3V")
+		(at 154.94 88.9 0)
+		(unit 1)
+		(exclude_from_sim no)
+		(in_bom yes)
+		(on_board yes)
+		(dnp no)
+		(fields_autoplaced yes)
+		(property "Reference" "#PWR023"
+			(at 154.94 92.71 0)
+			(effects
+				(font
+					(size 1.27 1.27)
+				)
+				(hide yes)
+			)
+		)
+		(property "Value" "+3.3V"
+			(at 154.94 83.82 0)
+			(effects
+				(font
+					(size 1.27 1.27)
+				)
+			)
+		)
+		(property "Footprint" ""
+			(at 154.94 88.9 0)
+			(effects
+				(font
+					(size 1.27 1.27)
+				)
+				(hide yes)
+			)
+		)
+		(property "Datasheet" ""
+			(at 154.94 88.9 0)
+			(effects
+				(font
+					(size 1.27 1.27)
+				)
+				(hide yes)
+			)
+		)
+		(property "Description" "Power symbol creates a global label with name \"+3.3V\""
+			(at 154.94 88.9 0)
+			(effects
+				(font
+					(size 1.27 1.27)
+				)
+				(hide yes)
+			)
+		)
+		(pin "1"
+		)
+		(instances
+			(project ""
+				(path "/210be09d-86cd-4faa-bb91-cc54c5972517/8074907f-d1dc-4b1d-805f-91e9bac82bf7"
+					(reference "#PWR023")
 					(unit 1)
 				)
@@
 		(dnp no)
 		(fields_autoplaced yes)
-		(property "Reference" "#PWR?"
+		(property "Reference" "#PWR0115"
 			(at 137.16 66.04 0)
 			(effects
@@
 			(project "projet electronique PCBot"
 				(path "/210be09d-86cd-4faa-bb91-cc54c5972517/8074907f-d1dc-4b1d-805f-91e9bac82bf7"
-					(reference "#PWR?")
+					(reference "#PWR0115")
 					(unit 1)
 				)
@@
 		(dnp no)
 		(fields_autoplaced yes)
-		(property "Reference" "J?"
+		(property "Reference" "J10"
 			(at 191.135 85.09 0)
 			(effects
@@
 			)
 		)
-		(property "Footprint" ""
+		(property "Footprint" "Connector_JST:JST_XH_B2B-XH-A_1x02_P2.50mm_Vertical"
 			(at 190.5 90.17 0)
 			(effects
@@
 			(project "projet electronique PCBot"
 				(path "/210be09d-86cd-4faa-bb91-cc54c5972517/8074907f-d1dc-4b1d-805f-91e9bac82bf7"
-					(reference "J?")
+					(reference "J10")
 					(unit 1)
 				)
@@
 		(dnp no)
 		(fields_autoplaced yes)
-		(property "Reference" "R?"
+		(property "Reference" "R11"
 			(at 107.95 91.4399 0)
 			(effects
@@
 			)
 		)
-		(property "Footprint" ""
+		(property "Footprint" "Resistor_SMD:R_0402_1005Metric"
 			(at 105.41 92.71 0)
 			(effects
@@
 			(project "projet electronique PCBot"
 				(path "/210be09d-86cd-4faa-bb91-cc54c5972517/8074907f-d1dc-4b1d-805f-91e9bac82bf7"
-					(reference "R?")
+					(reference "R11")
 					(unit 1)
 				)
@@
 		(dnp no)
 		(fields_autoplaced yes)
-		(property "Reference" "C?"
+		(property "Reference" "C20"
 			(at 172.72 64.7762 0)
 			(effects
@@
 			)
 		)
-		(property "Footprint" ""
+		(property "Footprint" "Capacitor_SMD:C_0805_2012Metric"
 			(at 170.18 66.04 0)
 			(effects
@@
 			(project "projet electronique PCBot"
 				(path "/210be09d-86cd-4faa-bb91-cc54c5972517/8074907f-d1dc-4b1d-805f-91e9bac82bf7"
-					(reference "C?")
+					(reference "C20")
 					(unit 1)
 				)
@@
 		(on_board yes)
 		(dnp no)
-		(property "Reference" "C?"
+		(property "Reference" "C18"
 			(at 110.4962 58.42 0)
 			(effects
@@
 			)
 		)
-		(property "Footprint" ""
+		(property "Footprint" "Capacitor_SMD:C_0402_1005Metric"
 			(at 111.76 60.96 0)
 			(effects
@@
 			(project "projet electronique PCBot"
 				(path "/210be09d-86cd-4faa-bb91-cc54c5972517/8074907f-d1dc-4b1d-805f-91e9bac82bf7"
-					(reference "C?")
+					(reference "C18")
 					(unit 1)
 				)
@@
 		(dnp no)
 		(fields_autoplaced yes)
-		(property "Reference" "#PWR?"
+		(property "Reference" "#PWR0114"
 			(at 116.84 138.43 0)
 			(effects
@@
 			(project "projet electronique PCBot"
 				(path "/210be09d-86cd-4faa-bb91-cc54c5972517/8074907f-d1dc-4b1d-805f-91e9bac82bf7"
-					(reference "#PWR?")
+					(reference "#PWR0114")
 					(unit 1)
 				)
@@
 		(dnp no)
 		(fields_autoplaced yes)
-		(property "Reference" "#PWR?"
+		(property "Reference" "#PWR0113"
 			(at 105.41 83.82 0)
 			(effects
@@
 			(project "projet electronique PCBot"
 				(path "/210be09d-86cd-4faa-bb91-cc54c5972517/8074907f-d1dc-4b1d-805f-91e9bac82bf7"
-					(reference "#PWR?")
+					(reference "#PWR0113")
 					(unit 1)
 				)
@@
 		(on_board yes)
 		(dnp no)
-		(property "Reference" "R?"
+		(property "Reference" "R12"
 			(at 139.7 77.4699 0)
 			(effects
@@
 			)
 		)
-		(property "Footprint" ""
+		(property "Footprint" "Resistor_SMD:R_0402_1005Metric"
 			(at 137.16 78.74 0)
 			(effects
@@
 			(project "projet electronique PCBot"
 				(path "/210be09d-86cd-4faa-bb91-cc54c5972517/8074907f-d1dc-4b1d-805f-91e9bac82bf7"
-					(reference "R?")
+					(reference "R12")
 					(unit 1)
 				)
@@
 			)
 		)
-		(property "Value" "DRV8833PWP"
+		(property "Value" "DRV8411APWPR"
 			(at 136.5759 123.19 0)
 			(effects
@@
 		(dnp no)
 		(fields_autoplaced yes)
-		(property "Reference" "R?"
+		(property "Reference" "R13"
 			(at 157.48 93.9799 0)
 			(effects
@@
 			)
 		)
-		(property "Footprint" ""
+		(property "Footprint" "Resistor_SMD:R_0402_1005Metric"
 			(at 154.94 95.25 0)
 			(effects
@@
 			(project "projet electronique PCBot"
 				(path "/210be09d-86cd-4faa-bb91-cc54c5972517/8074907f-d1dc-4b1d-805f-91e9bac82bf7"
-					(reference "R?")
+					(reference "R13")
 					(unit 1)
 				)
@@
 		(dnp no)
 		(fields_autoplaced yes)
-		(property "Reference" "#PWR?"
+		(property "Reference" "#PWR0116"
 			(at 100.33 60.96 0)
 			(effects
@@
 			(project "projet electronique PCBot"
 				(path "/210be09d-86cd-4faa-bb91-cc54c5972517/8074907f-d1dc-4b1d-805f-91e9bac82bf7"
-					(reference "#PWR?")
+					(reference "#PWR0116")
 					(unit 1)
 				)
@@
 		(dnp no)
 		(fields_autoplaced yes)
-		(property "Reference" "#PWR?"
+		(property "Reference" "#PWR0117"
 			(at 118.11 64.77 0)
 			(effects
@@
 			(project "projet electronique PCBot"
 				(path "/210be09d-86cd-4faa-bb91-cc54c5972517/8074907f-d1dc-4b1d-805f-91e9bac82bf7"
-					(reference "#PWR?")
-					(unit 1)
-				)
+					(reference "#PWR0117")
+					(unit 1)
+				)

Commit message: modif après revu prof
Connections:
- net TIM1_CH1: now also U4.16 (AIN1)
- net TIM1_CH1N: now also U4.15 (AIN2)
- net TIM1_CH2: now also U4.9 (BIN1)
- net TIM1_CH2N: now also U4.10 (BIN2)
- net PA4 renamed nFAULT
Changed lines of the file:
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@@
 		)
 	)
-	(hierarchical_label "PA4"
+	(hierarchical_label "nFAULT"
 		(shape input)
 		(at 158.75 102.87 0)
@@
 	(hierarchical_label "TIM1_CH1"
 		(shape input)
-		(at 102.87 106.68 0)
+		(at 119.38 107.95 180)
 		(effects
 			(font
 				(size 1.27 1.27)
 			)
-			(justify left)
+			(justify right)
 		)
 	)
 	(hierarchical_label "TIM1_CH2"
 		(shape input)
-		(at 102.87 109.22 0)
+		(at 119.38 113.03 180)
 		(effects
 			(font
 				(size 1.27 1.27)
 			)
-			(justify left)
+			(justify right)
 		)
 	)
@@
 	(hierarchical_label "TIM1_CH2N"
 		(shape input)
-		(at 102.87 116.84 0)
+		(at 119.38 115.57 180)
 		(effects
 			(font
 				(size 1.27 1.27)
 			)
-			(justify left)
+			(justify right)
 		)
 	)
 	(hierarchical_label "TIM1_CH1N"
 		(shape input)
-		(at 102.87 114.3 0)
+		(at 119.38 110.49 180)
 		(effects
 			(font
 				(size 1.27 1.27)
 			)
-			(justify left)
+			(justify right)
 		)
 	)

Commit message: suite placement composants
Connections:
- net at J9.1 (Pin_1): now also U4.5 (BOUT2); no longer U4.7 (BOUT1)
- net at J9.2 (Pin_2): now also U4.7 (BOUT1); no longer U4.5 (BOUT2)
Other:
- moved on the sheet: J9
Changed lines of the file:
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@@
 	(symbol
 		(lib_id "Connector:Conn_01x02_Pin")
-		(at 187.96 111.76 0)
+		(at 198.12 114.3 180)
 		(unit 1)
 		(exclude_from_sim no)
@@
 		(fields_autoplaced yes)
 		(property "Reference" "J9"
-			(at 188.595 106.68 0)
+			(at 199.39 111.7599 0)
 			(effects
 				(font
 					(size 1.27 1.27)
 				)
+				(justify right)
 			)
 		)
 		(property "Value" "Conn_01x02_Pin"
-			(at 188.595 109.22 0)
+			(at 199.39 114.2999 0)
 			(effects
 				(font
 					(size 1.27 1.27)
 				)
+				(justify right)
 			)
 		)
 		(property "Footprint" "Connector_JST:JST_XH_B2B-XH-A_1x02_P2.50mm_Vertical"
-			(at 187.96 111.76 0)
+			(at 198.12 114.3 0)
 			(effects
 				(font
@@
 		)
 		(property "Datasheet" "~"
-			(at 187.96 111.76 0)
+			(at 198.12 114.3 0)
 			(effects
 				(font
@@
 		)
 		(property "Description" "Generic connector, single row, 01x02, script generated"
-			(at 187.96 111.76 0)
+			(at 198.12 114.3 0)
 			(effects
 				(font

Commit message: modif routage fin
Connections:
- net BOUT2: now reaches J9.1 (Pin_1), U4.5 (BOUT2)
- net BOUT1: now reaches J9.2 (Pin_2), U4.7 (BOUT1)
- net AOUT1: now reaches J10.1 (Pin_1), U4.2 (AOUT1)
- net AOUT2: now reaches J10.2 (Pin_2), U4.4 (AOUT2)
Changed lines of the file:
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@@
+		)
+	)
+	(label "AOUT2"
+		(at 151.13 110.49 0)
+		(effects
+			(font
+				(size 1.27 1.27)
+			)
+			(justify left bottom)
+		)
+	)
+	(label "BOUT2"
+		(at 151.13 115.57 0)
+		(effects
+			(font
+				(size 1.27 1.27)
+			)
+			(justify left bottom)
+		)
+	)
+	(label "AOUT1"
+		(at 151.13 107.95 0)
+		(effects
+			(font
+				(size 1.27 1.27)
+			)
+			(justify left bottom)
+		)
+	)
+	(label "BOUT1"
+		(at 151.13 113.03 0)
+		(effects
+			(font
+				(size 1.27 1.27)
+			)
+			(justify left bottom)
 		)
 	)
