File: projet electronique PCBot/gestion_energie.kicad_sch (KiCad schematic)
At the start: 24 parts, among them J1 Conn_01x02_Pin, U1 BU33SD5WG-TR, U2 BQ25896RTWR

Commit message: grosse modif pcb du prof
Parts:
- removed R3: 10k, symbol Device:R_Small
- added J7: ON SWITCH, Connector_PinHeader_2.54mm:PinHeader_1x02_P2.54mm_Vertical, symbol Connector_Generic:Conn_01x02
- added JP1, JP2: SolderJumper_2_Open, Jumper:SolderJumper-2_P1.3mm_Open_TrianglePad1.0x1.5mm, symbol Jumper:SolderJumper_2_Open
- C10: renamed from C4; footprint (none) -> Capacitor_SMD:C_0402_1005Metric
- C11: renamed from C2; footprint (none) -> Capacitor_SMD:C_0603_1608Metric
- C12: renamed from C5; footprint (none) -> Capacitor_SMD:C_0603_1608Metric
- C13: renamed from C6; footprint (none) -> Capacitor_SMD:C_0603_1608Metric
- C14: renamed from C3; footprint (none) -> Capacitor_SMD:C_0402_1005Metric
- C15: renamed from C7; footprint (none) -> Capacitor_SMD:C_0603_1608Metric
- C16: renamed from C8; footprint (none) -> Capacitor_SMD:C_0402_1005Metric
- C17: renamed from C9; footprint (none) -> Capacitor_SMD:C_0402_1005Metric
- C9: renamed from C1; footprint (none) -> Capacitor_SMD:C_0402_1005Metric
- J8: renamed from J1; footprint (none) -> Connector_JST:JST_XH_B2B-XH-A_1x02_P2.50mm_Vertical
- L1: footprint (none) -> Inductor_SMD:L_1008_2520Metric
- R10: renamed from R2; value 30k1 -> 10k; footprint (none) -> Resistor_SMD:R_0402_1005Metric
- R3, R4: value R_Small -> 1k; footprint (none) -> Resistor_SMD:R_0402_1005Metric
- R5, R6: footprint (none) -> Resistor_SMD:R_0402_1005Metric
- R7: renamed from R4; value 260 -> 270R; footprint (none) -> Resistor_SMD:R_0402_1005Metric
- R8: renamed from R7; footprint (none) -> Resistor_SMD:R_0402_1005Metric
- R9: renamed from R1; value 5k23 -> 10k; footprint (none) -> Resistor_SMD:R_0402_1005Metric
- U2: footprint Package_DFN_QFN:Texas_S-PWQFN-N24_EP2.7x2.7mm_ThermalVias -> Package_DFN_QFN:Texas_RTW_WQFN-24-1EP_4x4mm_P0.5mm_EP2.7x2.7mm
- renumbered U1 to U3
Connections:
- net Earth is gone; now on net GND: C11.1, C12.2, C13.2, C14.2, C15.2, C16.2, C9.2, J8.2 (Pin_2), R10.2, R7.1, U2.17 (PGND), U2.18 (PGND), U2.2 (PSEL), U2.25 (PGND), U3.2 (GND)
- net +3.3V: now also U3.5 (VOUT)
- net SYS: now also JP2.2 (B); no longer C12.1, C13.1, L1.2, U2.15 (SYS), U2.16 (SYS)
- net VBUS: now also JP1.1 (A); no longer C9.1, U2.1 (VBUS)
- net GND: now reaches C17.2
- net GND: now also J7.1 (Pin_1); no longer U3.5 (VOUT)
- net at U2.12 (~{QON}): now also J7.2 (Pin_2)
- new net: C9.1, JP1.2 (B), U2.1 (VBUS)
- new net: C12.1, C13.1, JP2.1 (A), L1.2, U2.15 (SYS), U2.16 (SYS)
- no-connect marks 1 -> 0
Other:
- note removed: "A vérifier"
- moved on the sheet: C17

Commit message: suite placement composants
Connections:
- net +3.3V: now also R5.1, R6.1, R8.1
- net SW: now reaches C10.1, L1.1, U2.19 (SW), U2.20 (SW)
Other:
- note removed: "valeur des condensateurs a re vérifier auprès du prof"
Changed lines of the file:
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@@
-		)
-	)
-	(text "valeur des condensateurs a re vérifier auprès du prof\n"
-		(exclude_from_sim no)
-		(at 238.76 140.208 0)
-		(effects
-			(font
-				(size 1.27 1.27)
-			)
 		)
 	)
@@
 		(color 0 0 0 0)
 	)
+	(junction
+		(at 41.91 88.9)
+		(diameter 0)
+		(color 0 0 0 0)
+	)
 	(wire
 		(pts
@@
 	(wire
 		(pts
+			(xy 41.91 87.63) (xy 41.91 88.9)
+		)
+		(stroke
+			(width 0)
+			(type default)
+		)
+	)
+	(wire
+		(pts
 			(xy 228.6 124.46) (xy 226.06 124.46)
 		)
@@
 			(width 0)
 			(type default)
+		)
+	)
+	(label "SW"
+		(at 119.38 78.74 0)
+		(effects
+			(font
+				(size 1.27 1.27)
+			)
+			(justify left bottom)
 		)
 	)
@@
 					(unit 1)
 				)
+			)
+		)
+	)
+	(symbol
+		(lib_id "power:+3.3V")
+		(at 41.91 87.63 0)
+		(unit 1)
+		(exclude_from_sim no)
+		(in_bom yes)
+		(on_board yes)
+		(dnp no)
+		(fields_autoplaced yes)
+		(property "Reference" "#PWR0124"
+			(at 41.91 91.44 0)
+			(effects
+				(font
+					(size 1.27 1.27)
+				)
+				(hide yes)
+			)
+		)
+		(property "Value" "+3.3V"
+			(at 41.91 83.82 0)
+			(effects
+				(font
+					(size 1.27 1.27)
+				)
+			)
+		)
+		(property "Footprint" ""
+			(at 41.91 87.63 0)
+			(effects
+				(font
+					(size 1.27 1.27)
+				)
+				(hide yes)
+			)
+		)
+		(property "Datasheet" ""
+			(at 41.91 87.63 0)
+			(effects
+				(font
+					(size 1.27 1.27)
+				)
+				(hide yes)
+			)
+		)
+		(property "Description" ""
+			(at 41.91 87.63 0)
+			(effects
+				(font
+					(size 1.27 1.27)
+				)
+			)
+		)
+		(pin "1"
+		)
+		(instances
+			(project "projet electronique PCBot"
+				(path "/210be09d-86cd-4faa-bb91-cc54c5972517/d457b8fa-dc83-43ee-b672-fc417651a09a"
+					(reference "#PWR0124")
+					(unit 1)
+				)

Commit message: modif routage fin
Connections:
- net VBUS_TO_BQ: now reaches C9.1, JP1.2 (B), U2.1 (VBUS)
Changed lines of the file:
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@@
+		)
+	)
+	(label "VBUS_TO_BQ"
+		(at 78.74 73.66 0)
+		(effects
+			(font
+				(size 1.27 1.27)
+			)
+			(justify left bottom)
 		)
 	)
